Commit message: vids

File: mani_skill/assets/robot/panda/float_panda.urdf (robot description, URDF)
Before this commit: robot panda, 12 links, 11 joints
Links:
- link panda_hand: geometry collision mesh filename=franka_description/meshes/collision/hand.stl
- link panda_leftfinger: geometry collision box size=0.017088 0.01466 0.017088; collision box size=0.020466 0.015156 0.01515
- link panda_rightfinger: geometry collision box size=0.017088 0.01466 0.017088; collision box size=0.020466 0.015156 0.01515

File: mani_skill/assets/robot/panda/float_panda_correct_ori.urdf (robot description, URDF)
Before this commit: robot panda, 12 links, 11 joints
Links:
- link panda_hand: geometry collision mesh filename=franka_description/meshes/collision/hand.stl
- link panda_leftfinger: geometry collision box size=0.017088 0.01466 0.017088; collision box size=0.020466 0.015156 0.01515
- link panda_rightfinger: geometry collision box size=0.017088 0.01466 0.017088; collision box size=0.020466 0.015156 0.01515
